Commit message: adjusted inertial parameters of link_ee in iiwa14 description file

File: lbr_description/urdf/iiwa14/iiwa14_description.xacro (robot description, xacro)
@@ -252,7 +252,7 @@
         <link name="${robot_name}_link_ee">
             <inertial>
-                <origin rpy="0 0 0" xyz="0.01724 0.00679 0.02427" />
-                <mass value="0.412" />
-                <inertia ixx="0.000035" ixy="0.00000" ixz="0.00000" iyy="0.000035" iyz="0.0000" izz="0.000035" />
+                <origin rpy="0 0 0" xyz="0.018174 0.007152 0.023301" />
+                <mass value="0.390933" />
+                <inertia ixx="0.000299" ixy="-0.000149" ixz="-0.000028" iyy="0.000547" iyz="-0.000013" izz="0.000667" />
             </inertial>
             <visual>

Commit message: updated eef inertial parameters as the initial estimate was based on incorrect positioning of the camera wrt to the mounting bracket

File: lbr_description/urdf/iiwa14/iiwa14_description.xacro (robot description, xacro)
@@ -252,7 +252,7 @@
         <link name="${robot_name}_link_ee">
             <inertial>
-                <origin rpy="0 0 0" xyz="0.018174 0.007152 0.023301" />
-                <mass value="0.390933" />
-                <inertia ixx="0.000299" ixy="-0.000149" ixz="-0.000028" iyy="0.000547" iyz="-0.000013" izz="0.000667" />
+                <origin rpy="0 0 0" xyz="0.01823 0.00402 0.02330" />
+                <mass value="0.39127" />
+                <inertia ixx="0.00025" ixy="0.00000" ixz="0.00000" iyy="0.00055" iyz="0.00000" izz="0.00062" />
             </inertial>
             <visual>

Commit message: deleted eef from urdf and is  instead attached modularly in another bringup

File: lbr_description/urdf/iiwa14/iiwa14_description.xacro (robot description, xacro)
@@ -251,25 +251,4 @@
         </joint>
         <link name="${robot_name}_link_ee">
-            <inertial>
-                <origin rpy="0 0 0" xyz="0.01823 0.00402 0.02330" />
-                <mass value="0.39127" />
-                <inertia ixx="0.00025" ixy="0.00000" ixz="0.00000" iyy="0.00055" iyz="0.00000" izz="0.00062" />
-            </inertial>
-            <visual>
-                <origin rpy="0 0 0" xyz="0.0 0.0 0.0"/>
-                <geometry>
-                    <mesh filename="package://lbr_description/meshes/eefs/peg_eef_and_camera_assem.stl" />
-                </geometry>
-                <material name="custom_color">
-                    <color rgba="0.5 0.5 0.5 1.0"/>
-                </material>
-            </visual>
-        </link>
-        <joint name="${robot_name}_joint_tcp" type="fixed">
-            <parent link="${robot_name}_link_ee" />
-            <child link="${robot_name}_link_tcp" />
-            <origin xyz="0 0 0.0995" rpy="0 0 0" />
-        </joint>
-        <link name="${robot_name}_link_tcp">
         </link>
     </xacro:macro>

Commit message: assigned colours to robot mesh

File: lbr_description/urdf/iiwa14/iiwa14_description.xacro (robot description, xacro)
@@ -22,4 +22,16 @@
             joint_limits="${joint_limits}"
             system_config_path="${system_config_path}" />
+        <material name="orange">
+            <color rgba="0.949 0.360 0.098 1.0"/>
+        </material>
+        <material name="black">
+            <color rgba="0. 0. 0. 1.0"/>
+        </material>
+        <material name="grey">
+            <color rgba="0.7 0.7 0.7 1.0"/>
+        </material>
+        <material name="light_grey">
+            <color rgba="0.87 0.87 0.87 1.0"/>
+        </material>
         <link name="${robot_name}_link_0">
             <inertial>
@@ -33,4 +45,5 @@
                     <mesh filename="package://lbr_description/meshes/iiwa14/mjctrl_mesh/link_0.obj" />
                 </geometry>
+                <material name="grey"/>
             </visual>
         </link>
@@ -58,4 +71,5 @@
                     <mesh filename="package://lbr_description/meshes/iiwa14/mjctrl_mesh/link_1.obj" />
                 </geometry>
+                <material name="grey"/>
             </visual>
         </link>
@@ -83,4 +97,5 @@
                     <mesh filename="package://lbr_description/meshes/iiwa14/mjctrl_mesh/link_2_grey.obj" />
                 </geometry>
+                <material name="grey"/>
             </visual>
             <visual>
@@ -88,4 +103,5 @@
                     <mesh filename="package://lbr_description/meshes/iiwa14/mjctrl_mesh/link_2_orange.obj" />
                 </geometry>
+                <material name="orange"/>
             </visual>
         </link>
@@ -113,4 +129,5 @@
                     <mesh filename="package://lbr_description/meshes/iiwa14/mjctrl_mesh/link_3.obj" />
                 </geometry>
+                <material name="grey"/>
             </visual>
             <visual>
@@ -118,4 +135,5 @@
                     <mesh filename="package://lbr_description/meshes/iiwa14/mjctrl_mesh/band.obj" />
                 </geometry>
+                <material name="light_grey"/>
             </visual>
             <visual>
@@ -123,4 +141,5 @@
                     <mesh filename="package://lbr_description/meshes/iiwa14/mjctrl_mesh/kuka.obj" />
                 </geometry>
+                <material name="black"/>
             </visual>
         </link>
@@ -148,4 +167,5 @@
                     <mesh filename="package://lbr_description/meshes/iiwa14/mjctrl_mesh/link_4_orange.obj" />
                 </geometry>
+                <material name="orange"/>
             </visual>
             <visual>
@@ -153,4 +173,5 @@
                     <mesh filename="package://lbr_description/meshes/iiwa14/mjctrl_mesh/link_4_grey.obj" />
                 </geometry>
+                <material name="grey"/>
             </visual>
         </link>
@@ -178,4 +199,5 @@
                     <mesh filename="package://lbr_description/meshes/iiwa14/mjctrl_mesh/link_5.obj" />
                 </geometry>
+                <material name="grey"/>
             </visual>
             <visual>
@@ -183,4 +205,5 @@
                     <mesh filename="package://lbr_description/meshes/iiwa14/mjctrl_mesh/band.obj" />
                 </geometry>
+                <material name="light_grey"/>
             </visual>
             <visual>
@@ -188,4 +211,5 @@
                     <mesh filename="package://lbr_description/meshes/iiwa14/mjctrl_mesh/kuka.obj" />
                 </geometry>
+                <material name="black"/>
             </visual>
         </link>
@@ -213,4 +237,5 @@
                     <mesh filename="package://lbr_description/meshes/iiwa14/mjctrl_mesh/link_6_orange.obj" />
                 </geometry>
+                <material name="orange"/>
             </visual>
             <visual>
@@ -218,4 +243,5 @@
                     <mesh filename="package://lbr_description/meshes/iiwa14/mjctrl_mesh/link_6_grey.obj" />
                 </geometry>
+                <material name="grey"/>
             </visual>
         </link>
@@ -243,4 +269,5 @@
                     <mesh filename="package://lbr_description/meshes/iiwa14/mjctrl_mesh/link_7.obj" />
                 </geometry>
+                <material name="grey"/>
             </visual>
         </link>
